File: schema/schema.kicad_sch (KiCad schematic)
At the start: 0 parts

Commit message: Ver 1
Parts:
- added R1, R2: 5.1K, Resistor_SMD:R_1206_3216Metric, symbol Device:R
- added SW1: SW_Push, Button_Switch_THT:SW_PUSH_6mm_H5mm, symbol Switch:SW_Push
- added U1: WEMOS_D1_mini, RF_Module:WEMOS_D1_mini_light, symbol RF_Module:WEMOS_D1_mini
- added U2: ER_OLEDM0.91_1x-I2C, Display:ER_OLEDM0.91_1x-I2C, symbol Display_Graphic:ER_OLEDM0.91_1x-I2C
- added U3: (no value), ens160+aht21:ENS160+AHT21, symbol esn160+aht21:esn160+aht21
- added U4: (no value), ens160+aht21:18650 Battery Shield v3, symbol esn160+aht21:18650_battery_shield
Connections:
- new net +3.3V: R1.1, R2.1, U1.8 (3V3), U2.2 (VCC), U3.7 (3V3), U4.1 (3V)
- new net GND: U1.10 (GND), U2.1 (GND), U3.6 (GND), U4.2 (GND)
- new net SCL: R1.2, U1.14 (SCL/D1), U2.3 (SCL), U3.5 (SCL/SCLK)
- new net SDA: R2.2, U1.13 (SDA/D2), U2.4 (SDA), U3.4 (SDA/MOSI)
- new net button_in: SW1.1, U1.5 (MISO/D6)
- new net button_out: SW1.2, U1.4 (SCK/D5)
- no-connect marks 0 -> 15
